File: Hardware/Qwiic MP3 Trigger.brd (EAGLE design)
At the start: 25.4 x 50.8 mm, 104 parts, among them J1 MICRO-SD, J3 PTH, J7 ISP, J8 3.5mm Audio, J9 Poke-Home, U1 TPA2005D1, U2 WT2003S, U3 AP2112-3.3V, U4 ATTINY84-ARDUINO

Commit message: Modify RCs on amp input to match impedance. Should reduce pop and gain a bit.
Parts:
- C5: value 1.0uF -> 22nF
- C7, C8: value 0.1uF -> 10nF
- R11: value 100k -> 47k
- R5, R9: value 10k -> 100k
Changed lines of the file:
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@@
 <?xml version="1.0" encoding="utf-8"?>
 <!DOCTYPE eagle SYSTEM "eagle.dtd">
-<eagle version="9.2.1">
+<eagle version="9.6.0">
 <drawing>
 <settings>
@@
 <layer number="44" name="Drills" color="7" fill="1" visible="no" active="yes"/>
 <layer number="45" name="Holes" color="7" fill="1" visible="yes" active="yes"/>
-<layer number="46" name="Milling" color="3" fill="1" visible="yes" active="yes"/>
+<layer number="46" name="Milling" color="3" fill="1" visible="no" active="yes"/>
 <layer number="47" name="Measures" color="7" fill="1" visible="no" active="yes"/>
 <layer number="48" name="Document" color="7" fill="1" visible="no" active="yes"/>
@@
 <layer number="95" name="Names" color="7" fill="1" visible="no" active="no"/>
 <layer number="96" name="Values" color="7" fill="1" visible="no" active="no"/>
-<layer number="2" name="Route2" color="1" fill="3" visible="yes" active="yes"/>
-<layer number="15" name="Route15" color="4" fill="6" visible="yes" active="yes"/>
+<layer number="2" name="Route2" color="1" fill="3" visible="no" active="yes"/>
+<layer number="15" name="Route15" color="4" fill="6" visible="no" active="yes"/>
 <layer number="3" name="Route3" color="4" fill="3" visible="no" active="no"/>
 <layer number="4" name="Route4" color="1" fill="4" visible="no" active="no"/>
@@
 <layer number="115" name="ReferenceISLANDS" color="7" fill="1" visible="no" active="no"/>
 <layer number="116" name="Patch_BOT" color="9" fill="4" visible="no" active="no"/>
+<layer number="117" name="PM_Ref" color="7" fill="1" visible="no" active="no"/>
 <layer number="118" name="Rect_Pads" color="7" fill="1" visible="no" active="no"/>
+<layer number="119" name="PF_Ref" color="7" fill="1" visible="no" active="no"/>
+<layer number="120" name="WFL_Ref" color="7" fill="1" visible="no" active="no"/>
 <layer number="121" name="_tsilk" color="7" fill="1" visible="no" active="no"/>
 <layer number="122" name="_bsilk" color="7" fill="1" visible="no" active="no"/>
@@
 <attribute name="VALUE" value="10k" x="22.86" y="29.591" size="1.778" layer="27" rot="R180" display="off"/>
 </element>
-<element name="R11" library="SparkFun-Resistors" package="0603" value="100k" x="22.86" y="33.02" smashed="yes" rot="R180">
+<element name="R11" library="SparkFun-Resistors" package="0603" value="47k" x="22.86" y="33.02" smashed="yes" rot="R180">
 <attribute name="NAME" x="22.86" y="32.258" size="0.6096" layer="25" font="vector" ratio="20" rot="R180" align="bottom-center"/>
-<attribute name="PROD_ID" value="RES-07828" x="22.86" y="33.02" size="1.778" layer="27" rot="R180" display="off"/>
-<attribute name="VALUE" value="100k" x="25.4" y="32.766" size="0.6096" layer="27" font="vector" ratio="20" rot="R180" align="top-center"/>
+<attribute name="PROD_ID" value="RES-07871" x="22.86" y="33.02" size="1.778" layer="27" rot="R180" display="off"/>
+<attribute name="VALUE" value="47k" x="25.4" y="32.766" size="0.6096" layer="27" font="vector" ratio="20" rot="R180" align="top-center"/>
 <attribute name="VALUE" value="4.7k" x="22.86" y="33.02" size="1.778" layer="27" rot="R180" display="off"/>
 </element>
@@
 <attribute name="VALUE" x="7.493" y="8.636" size="0.6096" layer="27" font="vector" ratio="20" rot="R180" align="top-center"/>
 </element>
-<element name="R5" library="SparkFun-Resistors" package="0603" value="10k" x="22.86" y="34.544" smashed="yes" rot="R180">
+<element name="R5" library="SparkFun-Resistors" package="0603" value="100k" x="22.86" y="34.544" smashed="yes" rot="R180">
 <attribute name="NAME" x="22.86" y="33.782" size="0.6096" layer="25" font="vector" ratio="20" rot="R180" align="bottom-center"/>
-<attribute name="PROD_ID" value="RES-00824" x="22.86" y="34.544" size="1.778" layer="27" font="vector" ratio="15" rot="R180" display="off"/>
-<attribute name="VALUE" x="25.273" y="34.163" size="0.6096" layer="27" font="vector" ratio="20" rot="R180" align="top-center"/>
-</element>
-<element name="R9" library="SparkFun-Resistors" package="0603" value="10k" x="22.86" y="38.1" smashed="yes" rot="R180">
+<attribute name="PROD_ID" value="RES-07828" x="22.86" y="34.544" size="1.778" layer="27" font="vector" ratio="15" rot="R180" display="off"/>
+<attribute name="VALUE" value="100k" x="25.273" y="34.163" size="0.6096" layer="27" font="vector" ratio="20" rot="R180" align="top-center"/>
+</element>
+<element name="R9" library="SparkFun-Resistors" package="0603" value="100k" x="22.86" y="38.1" smashed="yes" rot="R180">
 <attribute name="NAME" x="22.86" y="37.338" size="0.6096" layer="25" font="vector" ratio="20" rot="R180" align="bottom-center"/>
-<attribute name="PROD_ID" value="RES-00824" x="22.86" y="38.1" size="1.778" layer="27" font="vector" ratio="15" rot="R180" display="off"/>
-<attribute name="VALUE" x="25.273" y="37.846" size="0.6096" layer="27" font="vector" ratio="20" rot="R180" align="top-center"/>
+<attribute name="PROD_ID" value="RES-07828" x="22.86" y="38.1" size="1.778" layer="27" font="vector" ratio="15" rot="R180" display="off"/>
+<attribute name="VALUE" value="100k" x="25.273" y="37.846" size="0.6096" layer="27" font="vector" ratio="20" rot="R180" align="top-center"/>
 </element>
 <element name="U1" library="SparkFun-IC-Amplifiers" package="QFN-8_PAD" value="TPA2005D1" x="19.05" y="31.75" smashed="yes" rot="R90">
@@
 <attribute name="VALUE" value="TPA2005D1" x="19.05" y="31.75" size="1.778" layer="27" rot="R90" display="off"/>
 </element>
-<element name="C7" library="SparkFun-Capacitors" package="0603" value="0.1uF" x="22.86" y="36.068" smashed="yes">
+<element name="C7" library="SparkFun-Capacitors" package="0603" value="10nF" x="22.86" y="36.068" smashed="yes">
 <attribute name="NAME" x="22.86" y="36.83" size="0.6096" layer="25" font="vector" ratio="20" align="bottom-center"/>
-<attribute name="PROD_ID" value="CAP-00810" x="22.86" y="36.068" size="1.778" layer="27" font="vector" ratio="15" display="off"/>
-<attribute name="VALUE" x="25.781" y="36.449" size="0.6096" layer="27" font="vector" ratio="20" align="top-center"/>
-</element>
-<element name="C8" library="SparkFun-Capacitors" package="0603" value="0.1uF" x="22.86" y="39.624" smashed="yes">
+<attribute name="PROD_ID" value="CAP-00867" x="22.86" y="36.068" size="1.778" layer="27" font="vector" ratio="15" display="off"/>
+<attribute name="VALUE" value="10nF" x="25.781" y="36.449" size="0.6096" layer="27" font="vector" ratio="20" align="top-center"/>
+</element>
+<element name="C8" library="SparkFun-Capacitors" package="0603" value="10nF" x="22.86" y="39.624" smashed="yes">
 <attribute name="NAME" x="22.86" y="40.386" size="0.6096" layer="25" font="vector" ratio="20" align="bottom-center"/>
-<attribute name="PROD_ID" value="CAP-00810" x="22.86" y="39.624" size="1.778" layer="27" font="vector" ratio="15" display="off"/>
-<attribute name="VALUE" x="25.908" y="40.005" size="0.6096" layer="27" font="vector" ratio="20" align="top-center"/>
+<attribute name="PROD_ID" value="CAP-00867" x="22.86" y="39.624" size="1.778" layer="27" font="vector" ratio="15" display="off"/>
+<attribute name="VALUE" value="10nF" x="25.908" y="40.005" size="0.6096" layer="27" font="vector" ratio="20" align="top-center"/>
 </element>
 <element name="J11" library="SparkFun-Connectors" package="1X04_NO_SILK" value="" x="16.51" y="49.53" smashed="yes" rot="R180">
@@
 <attribute name="VALUE" x="17.78" y="49.022" size="0.6096" layer="27" font="vector" ratio="20" rot="R180"/>
 </element>
-<element name="C5" library="SparkFun-Capacitors" package="0603" value="1.0uF" x="22.86" y="31.496" smashed="yes" rot="R180">
+<element name="C5" library="SparkFun-Capacitors" package="0603" value="22nF" x="22.86" y="31.496" smashed="yes" rot="R180">
 <attribute name="NAME" x="22.86" y="30.734" size="0.6096" layer="25" font="vector" ratio="20" rot="R180" align="bottom-center"/>
-<attribute name="PROD_ID" value="CAP-00868" x="22.86" y="31.496" size="1.778" layer="27" font="vector" ratio="15" rot="R180" display="off"/>
-<attribute name="VALUE" x="25.654" y="31.242" size="0.6096" layer="27" font="vector" ratio="20" rot="R180" align="top-center"/>
+<attribute name="PROD_ID" value="CAP-07885" x="22.86" y="31.496" size="1.778" layer="27" font="vector" ratio="15" rot="R180" display="off"/>
+<attribute name="VALUE" value="22nF" x="25.654" y="31.242" size="0.6096" layer="27" font="vector" ratio="20" rot="R180" align="top-center"/>
 </element>
 <element name="JP7" library="SparkFun-Jumpers" package="SMT-JUMPER_2_NO_SILK" value="ADR" x="13.97" y="25.4" smashed="yes" rot="R180">
