File: Hardware/Qwiic MP3 Trigger.sch (EAGLE design)
At the start: 57 parts, among them J1 MICRO-SD, J3 PTH, J7 ISP, J8 3.5mm Audio, J9 Poke-Home, U1 TPA2005D1, U2 WT2003S, U3 AP2112-3.3V, U4 ATTINY84-ARDUINO

Commit message: Modify RCs on amp input to match impedance. Should reduce pop and gain a bit.
Parts:
- C5: value 1.0uF -> 22nF; device SparkFun-Capacitors:1.0UF-0603-16V-10% -> SparkFun-Capacitors:22NF/22,000PF-0603-50V-10%
- C7, C8: value 0.1uF -> 10nF; device SparkFun-Capacitors:0.1UF-0603-25V-(+80/-20%) -> SparkFun-Capacitors:10NF-0603-50V-10%
- R11: value 100k -> 47k; device SparkFun-Resistors:100KOHM-0603-1/10W-1% -> SparkFun-Resistors:47KOHM-0603-1/10W-1%
- R5, R9: value 10k -> 100k; device SparkFun-Resistors:10KOHM-0603-1/10W-1% -> SparkFun-Resistors:100KOHM-0603-1/10W-1%

Commit message: Increment version number on sch
Other:
- note added: "v12"
- note removed: "X10"
Changed lines of the file:
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@@
 <plain>
 <text x="170.434" y="11.43" size="2.54" layer="94">N. Seidle</text>
-<text x="237.744" y="7.366" size="2.54" layer="94">X10</text>
+<text x="237.744" y="7.366" size="2.54" layer="94">v12</text>
 <text x="74.803" y="75.311" size="1.778" layer="97" rot="R90">Power</text>
 <text x="154.178" y="99.06" size="1.778" layer="97">7-Bit Unshifted I2C Address
